Commit message: Feature/gnss sensor (#21)
* added gnss sensor launch

* set zurich as testing location

* added realsense d455

* barcelona coordinates

---------

Co-authored-by: Paul Joseph <paul@bubble-robotics.com>

File: blue_description/description/bluerov2/config.xacro (robot description, xacro)
@@ -5,4 +5,5 @@
   <xacro:arg name="use_imu" default="true" />
   <xacro:arg name="use_dvl" default="true" />
+  <xacro:arg name="use_gnss" default="true" />
   <!-- Import BlueROV2 macro -->
   <xacro:include filename="$(find blue_description)/description/bluerov2/urdf.xacro" />

File: blue_description/description/bluerov2/gazebo.xacro (robot description, xacro)
@@ -5,4 +5,5 @@
     <xacro:arg name="use_imu" default="true" />
     <xacro:arg name="use_dvl" default="true" />
+    <xacro:arg name="use_gnss" default="true" />
     <gazebo>
       <plugin name="ArduPilotPlugin" filename="libArduPilotPlugin.so">
@@ -115,5 +116,5 @@
     <xacro:include filename="$(find blue_description)/description/bluerov2/sensors.xacro" />
     <xacro:sensors_macro prefix="$(arg prefix)" use_sim="true" use_imu="$(arg use_imu)"
-      use_dvl="$(arg use_dvl)" />
+      use_dvl="$(arg use_dvl)" use_gnss="$(arg use_gnss)" />
     <!-- Publish the ground-truth pose -->
     <gazebo>

File: blue_description/description/bluerov2/sensors.xacro (robot description, xacro)
@@ -1,5 +1,5 @@
 <?xml version="1.0"?>
 <robot xmlns:xacro="http://ros.org/wiki/xacro">
-  <xacro:macro name="sensors_macro" params="prefix:='' use_sim:=false use_imu:=true use_dvl:=true">
+  <xacro:macro name="sensors_macro" params="prefix:='' use_sim:=false use_imu:=true use_dvl:=true use_gnss:=true">
     <!-- Import IMU sensor -->
     <xacro:include filename="$(find blue_description)/description/vn100/urdf.xacro" />
@@ -14,15 +14,11 @@
       <origin rpy="3.1416 0 0" xyz="0.0 0.0 -0.12" />
     </xacro:dvl_urdf>
+    <!-- GNSS sensor -->
+    <xacro:include filename="$(find sensors_gnss)/description/ZED-F9P/urdf.xacro" />
+    <xacro:gnss_urdf prefix="$(arg prefix)" parent="$(arg prefix)base_link" />
     <!-- Import Realsense URDF-->
     <xacro:include filename="$(find sensors_camera)/description/d455/urdf.xacro" />
     <xacro:realsense_d455_urdf parent="$(arg prefix)base_link" prefix="$(arg prefix)">
     </xacro:realsense_d455_urdf>
-    <!-- TODO: eventually these should only be executed when a flag use_d455 is
-     set during launch. However, currently, parameter passing does not work, the
-     chain is broken at some link.-->
-    <xacro:include filename="$(find sensors_camera)/description/d455/gazebo.xacro"/>
-    <xacro:realsense_d455_gazebo reference="$(arg prefix)realsense_d455_link">
-    </xacro:realsense_d455_gazebo>
-    <!-- Import Realsense Sensor specificaitons-->
     <!-- Add Gazebo sensor plugins if in simulation -->
     <xacro:if value="$(arg use_sim)">
@@ -32,4 +28,11 @@
       <xacro:include filename="$(find blue_description)/description/dvl/gazebo.xacro" />
       <xacro:dvl_gazebo reference="$(arg prefix)dvl_link" topic="/dvl/data_test" />
+      <xacro:include filename="$(find sensors_gnss)/description/ZED-F9P/gazebo.xacro" />
+      <xacro:gnss_gazebo reference="$(arg prefix)gnss_link" />
+    <!-- TODO: eventually these should only be executed when a flag use_d455 is
+     set during launch. However, currently, parameter passing does not work, the
+     chain is broken at some link.-->
+      <xacro:include filename="$(find sensors_camera)/description/d455/gazebo.xacro" />
+      <xacro:realsense_d455_gazebo reference="$(arg prefix)realsense_d455_link"/>
     </xacro:if>
   </xacro:macro>
