Commit message: Added EGO planner obstacle avoidance test for MT

File: blue_description/description/bluerov2_heavy/urdf.xacro (robot description, xacro)
@@ -6,5 +6,5 @@
       <inertial>
         <origin rpy="0 0 0" xyz="0.0 0.0 0.011" />
-        <mass value="13.0" />
+        <mass value="13.15" />
         <inertia
           ixx="0.26"
@@ -43,4 +43,13 @@
         </fluid_added_mass>
       </inertial>
+    </gazebo>
+    <gazebo reference="${prefix}base_footprint">
+      <sensor name="contact_sensor" type="contact">
+        <always_on>true</always_on>
+        <update_rate>50</update_rate>
+        <contact>
+          <collision>base_footprint_fixed_joint_lump__base_link_collision_collision</collision>
+        </contact>
+      </sensor>
     </gazebo>
     <joint name="${prefix}base_footprint_joint" type="fixed">
